File: DSS3P.sch (EAGLE design)
At the start: 289 parts, among them J1 J5MM

Commit message: .
Parts:
- removed 3T1: TRANS_ER35/20/11, DSS:TRANS_ER35/20/11
- added U$2: TRANS_ER38, DSS0:TRANS_ER38
Connections:
- net GND: now also U$2.GND; no longer 3T1.P$4, 3T1.P$8
- net N$100: now also U$2.5-2; no longer 3T1.P$5
- net N$14: now also U$2.IN2; no longer 3T1.P$2
- net N$87: now also U$2.IN1; no longer 3T1.P$1
- net N$95: now also U$2.12-1; no longer 3T1.P$6
- net N$96: now also U$2.12-2; no longer 3T1.P$7
- net N$97: now also U$2.24-1; no longer 3T1.P$9
- net N$98: now also U$2.24-2; no longer 3T1.P$10
- net N$99: now also U$2.5-1; no longer 3T1.P$3

Commit message: .
Parts:
- 1R46: device resistor:R-EU_M0805 -> resistor:R-EU_R1206W
- 1R6: device resistor:R-EU_R1206W -> resistor:R-EU_R0805
Changed lines of the file:
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@@
 <grid distance="100" unitdist="mil" unit="mil" style="lines" multiple="1" display="yes" altdistance="0.01" altunitdist="inch" altunit="inch"/>
 <layers>
-<layer number="1" name="Top" color="4" fill="1" visible="no" active="no"/>
-<layer number="2" name="Route2" color="1" fill="3" visible="no" active="no"/>
-<layer number="3" name="Route3" color="4" fill="3" visible="no" active="no"/>
-<layer number="4" name="Route4" color="1" fill="4" visible="no" active="no"/>
-<layer number="5" name="Route5" color="4" fill="4" visible="no" active="no"/>
-<layer number="6" name="Route6" color="1" fill="8" visible="no" active="no"/>
-<layer number="7" name="Route7" color="4" fill="8" visible="no" active="no"/>
-<layer number="8" name="Route8" color="1" fill="2" visible="no" active="no"/>
-<layer number="9" name="Route9" color="4" fill="2" visible="no" active="no"/>
-<layer number="10" name="Route10" color="1" fill="7" visible="no" active="no"/>
-<layer number="11" name="Route11" color="4" fill="7" visible="no" active="no"/>
-<layer number="12" name="Route12" color="1" fill="5" visible="no" active="no"/>
-<layer number="13" name="Route13" color="4" fill="5" visible="no" active="no"/>
-<layer number="14" name="Route14" color="1" fill="6" visible="no" active="no"/>
-<layer number="15" name="Route15" color="4" fill="6" visible="no" active="no"/>
-<layer number="16" name="Bottom" color="1" fill="1" visible="no" active="no"/>
-<layer number="17" name="Pads" color="2" fill="1" visible="no" active="no"/>
-<layer number="18" name="Vias" color="2" fill="1" visible="no" active="no"/>
-<layer number="19" name="Unrouted" color="6" fill="1" visible="no" active="no"/>
-<layer number="20" name="Dimension" color="15" fill="1" visible="no" active="no"/>
-<layer number="21" name="tPlace" color="7" fill="1" visible="no" active="no"/>
-<layer number="22" name="bPlace" color="7" fill="1" visible="no" active="no"/>
-<layer number="23" name="tOrigins" color="15" fill="1" visible="no" active="no"/>
-<layer number="24" name="bOrigins" color="15" fill="1" visible="no" active="no"/>
-<layer number="25" name="tNames" color="7" fill="1" visible="no" active="no"/>
-<layer number="26" name="bNames" color="7" fill="1" visible="no" active="no"/>
-<layer number="27" name="tValues" color="7" fill="1" visible="no" active="no"/>
-<layer number="28" name="bValues" color="7" fill="1" visible="no" active="no"/>
+<layer number="1" name="Top" color="4" fill="1" visible="yes" active="no"/>
+<layer number="2" name="Route2" color="1" fill="3" visible="yes" active="no"/>
+<layer number="3" name="Route3" color="4" fill="3" visible="yes" active="no"/>
+<layer number="4" name="Route4" color="1" fill="4" visible="yes" active="no"/>
+<layer number="5" name="Route5" color="4" fill="4" visible="yes" active="no"/>
+<layer number="6" name="Route6" color="1" fill="8" visible="yes" active="no"/>
+<layer number="7" name="Route7" color="4" fill="8" visible="yes" active="no"/>
+<layer number="8" name="Route8" color="1" fill="2" visible="yes" active="no"/>
+<layer number="9" name="Route9" color="4" fill="2" visible="yes" active="no"/>
+<layer number="10" name="Route10" color="1" fill="7" visible="yes" active="no"/>
+<layer number="11" name="Route11" color="4" fill="7" visible="yes" active="no"/>
+<layer number="12" name="Route12" color="1" fill="5" visible="yes" active="no"/>
+<layer number="13" name="Route13" color="4" fill="5" visible="yes" active="no"/>
+<layer number="14" name="Route14" color="1" fill="6" visible="yes" active="no"/>
+<layer number="15" name="Route15" color="4" fill="6" visible="yes" active="no"/>
+<layer number="16" name="Bottom" color="1" fill="1" visible="yes" active="no"/>
+<layer number="17" name="Pads" color="2" fill="1" visible="yes" active="no"/>
+<layer number="18" name="Vias" color="2" fill="1" visible="yes" active="no"/>
+<layer number="19" name="Unrouted" color="6" fill="1" visible="yes" active="no"/>
+<layer number="20" name="Dimension" color="15" fill="1" visible="yes" active="no"/>
+<layer number="21" name="tPlace" color="7" fill="1" visible="yes" active="no"/>
+<layer number="22" name="bPlace" color="7" fill="1" visible="yes" active="no"/>
+<layer number="23" name="tOrigins" color="15" fill="1" visible="yes" active="no"/>
+<layer number="24" name="bOrigins" color="15" fill="1" visible="yes" active="no"/>
+<layer number="25" name="tNames" color="7" fill="1" visible="yes" active="no"/>
+<layer number="26" name="bNames" color="7" fill="1" visible="yes" active="no"/>
+<layer number="27" name="tValues" color="7" fill="1" visible="yes" active="no"/>
+<layer number="28" name="bValues" color="7" fill="1" visible="yes" active="no"/>
 <layer number="29" name="tStop" color="7" fill="3" visible="no" active="no"/>
 <layer number="30" name="bStop" color="7" fill="6" visible="no" active="no"/>
@@
 <layer number="35" name="tGlue" color="7" fill="4" visible="no" active="no"/>
 <layer number="36" name="bGlue" color="7" fill="5" visible="no" active="no"/>
-<layer number="37" name="tTest" color="7" fill="1" visible="no" active="no"/>
-<layer number="38" name="bTest" color="7" fill="1" visible="no" active="no"/>
+<layer number="37" name="tTest" color="7" fill="1" visible="yes" active="no"/>
+<layer number="38" name="bTest" color="7" fill="1" visible="yes" active="no"/>
 <layer number="39" name="tKeepout" color="4" fill="11" visible="no" active="no"/>
 <layer number="40" name="bKeepout" color="1" fill="11" visible="no" active="no"/>
@@
 <layer number="44" name="Drills" color="7" fill="1" visible="no" active="no"/>
 <layer number="45" name="Holes" color="7" fill="1" visible="no" active="no"/>
-<layer number="46" name="Milling" color="3" fill="1" visible="no" active="no"/>
-<layer number="47" name="Measures" color="7" fill="1" visible="no" active="no"/>
-<layer number="48" name="Document" color="7" fill="1" visible="no" active="no"/>
-<layer number="49" name="Reference" color="7" fill="1" visible="no" active="no"/>
-<layer number="50" name="dxf" color="7" fill="1" visible="no" active="no"/>
-<layer number="51" name="tDocu" color="7" fill="1" visible="no" active="no"/>
-<layer number="52" name="bDocu" color="7" fill="1" visible="no" active="no"/>
-<layer number="53" name="tGND_GNDA" color="7" fill="9" visible="no" active="no"/>
-<layer number="54" name="bGND_GNDA" color="1" fill="9" visible="no" active="no"/>
-<layer number="56" name="wert" color="7" fill="1" visible="no" active="no"/>
-<layer number="57" name="tCAD" color="7" fill="1" visible="no" active="no"/>
+<layer number="46" name="Milling" color="3" fill="1" visible="yes" active="no"/>
+<layer number="47" name="Measures" color="7" fill="1" visible="yes" active="no"/>
+<layer number="48" name="Document" color="7" fill="1" visible="yes" active="no"/>
+<layer number="49" name="Reference" color="7" fill="1" visible="yes" active="no"/>
+<layer number="50" name="dxf" color="7" fill="1" visible="yes" active="no"/>
+<layer number="51" name="tDocu" color="7" fill="1" visible="yes" active="no"/>
+<layer number="52" name="bDocu" color="7" fill="1" visible="yes" active="no"/>
+<layer number="53" name="tGND_GNDA" color="7" fill="9" visible="yes" active="no"/>
+<layer number="54" name="bGND_GNDA" color="1" fill="9" visible="yes" active="no"/>
+<layer number="56" name="wert" color="7" fill="1" visible="yes" active="no"/>
+<layer number="57" name="tCAD" color="7" fill="1" visible="yes" active="no"/>
 <layer number="90" name="Modules" color="5" fill="1" visible="yes" active="yes"/>
 <layer number="91" name="Nets" color="2" fill="1" visible="yes" active="yes"/>
@@
 <part name="1R2" library="resistor" deviceset="R-TRIMM" device="3296W" value="10k"/>
 <part name="1R10" library="resistor" deviceset="R-EU_" device="M1206" value="10k"/>
-<part name="1R6" library="resistor" deviceset="R-EU_" device="R1206W" value="1k"/>
-<part name="1R46" library="resistor" deviceset="R-EU_" device="M0805" value="100"/>
+<part name="1R6" library="resistor" deviceset="R-EU_" device="R0805" value="1k"/>
+<part name="1R46" library="resistor" deviceset="R-EU_" device="R1206W" value="100"/>
 <part name="P+28" library="supply1" deviceset="+5V" device=""/>
 <part name="P+29" library="supply1" deviceset="+24V" device=""/>
@@
 <instance part="1VT5" gate="A" x="281.94" y="25.4" smashed="yes">
 <attribute name="NAME" x="290.83" y="22.86" size="1.778" layer="95"/>
-<attribute name="VALUE" x="289.56" y="20.32" size="1.778" layer="96"/>
+<attribute name="VALUE" x="279.4" y="15.24" size="1.778" layer="96"/>
 </instance>
 <instance part="SOLDER1" gate="G$1" x="304.8" y="38.1" smashed="yes" rot="R270">
@@
 </instance>
 <instance part="1SJ9" gate="1" x="294.64" y="22.86" smashed="yes">
-<attribute name="NAME" x="290.83" y="19.05" size="1.778" layer="95"/>
+<attribute name="NAME" x="280.67" y="11.43" size="1.778" layer="95"/>
 <attribute name="VALUE" x="292.1" y="19.05" size="1.778" layer="96"/>
 </instance>

Commit message: .
Parts:
- 1R42, 1R45: device resistor:R-EU_0613/15 -> resistor:R-EU_0207/10
- 1R55: device resistor:R-EU_0204/7 -> resistor:R-EU_R1206W
- renumbered SV1 to FAN_C, SV3 to PREH_C
Changed lines of the file:
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@@
 <part name="1T3" library="ON Semiconductor_simistor" deviceset="BTA16-600CW3G" device="TO220DS" value="BTA12-600CWRG"/>
 <part name="1R35" library="resistor" deviceset="R-EU_" device="M0805" value="510"/>
-<part name="1R42" library="resistor" deviceset="R-EU_" device="0613/15" value="390"/>
+<part name="1R42" library="resistor" deviceset="R-EU_" device="0207/10" value="390"/>
 <part name="1R39" library="resistor" deviceset="R-EU_" device="0613/15" value="390"/>
-<part name="1R45" library="resistor" deviceset="R-EU_" device="0613/15" value="39"/>
+<part name="1R45" library="resistor" deviceset="R-EU_" device="0207/10" value="39"/>
 <part name="1C19" library="resistor" deviceset="C-EU" device="102-043X133" value="100nx400v"/>
 <part name="1OK1" library="DSS" deviceset="MOC3063M" device="D" value="MOC3063"/>
@@
 <part name="GND4" library="supply1" deviceset="GND" device=""/>
 <part name="SOLDER2" library="DSS0" deviceset="CON_DIN5" device=""/>
-<part name="1R55" library="resistor" deviceset="R-EU_" device="0204/7" value="3k"/>
+<part name="1R55" library="resistor" deviceset="R-EU_" device="R1206W" value="3k"/>
 <part name="1R8" library="resistor" deviceset="R-EU_" device="M0805" value="1k"/>
 <part name="1R38" library="resistor" deviceset="R-EU_" device="M1206" value="100"/>
@@
 <part name="1SJ3" library="jumper" deviceset="SJ" device=""/>
 <part name="1SJ9" library="jumper" deviceset="SJ" device=""/>
-<part name="SV1" library="con-lstb" deviceset="MA05-2" device=""/>
+<part name="FAN_C" library="con-lstb" deviceset="MA05-2" device=""/>
 <part name="PWFAN" library="con-wago-508" deviceset="W237-02P" device="">
 <attribute name="MF" value=""/>
@@
 <attribute name="OC_NEWARK" value="unknown"/>
 </part>
-<part name="SV3" library="con-lstb" deviceset="MA04-2" device=""/>
+<part name="PREH_C" library="con-lstb" deviceset="MA04-2" device=""/>
 <part name="PWFAN1" library="con-wago-508" deviceset="W237-02P" device="">
 <attribute name="MF" value=""/>
@@
 <attribute name="VALUE" x="292.1" y="19.05" size="1.778" layer="96"/>
 </instance>
-<instance part="SV1" gate="G$1" x="457.2" y="25.4"/>
+<instance part="FAN_C" gate="G$1" x="457.2" y="25.4"/>
 <instance part="PWFAN" gate="-1" x="482.6" y="-13.97" smashed="yes" rot="MR0">
 <attribute name="NAME" x="483.87" y="-13.081" size="1.778" layer="95" rot="MR180"/>
 </instance>
 <instance part="PWFAN" gate="-2" x="492.76" y="-22.86" rot="MR0"/>
-<instance part="SV3" gate="G$1" x="457.2" y="49.53"/>
+<instance part="PREH_C" gate="G$1" x="457.2" y="49.53"/>
 <instance part="PWFAN1" gate="-1" x="566.42" y="-12.7" rot="MR0"/>
 <instance part="PWFAN1" gate="-2" x="566.42" y="-17.78" rot="MR0"/>
@@
 </segment>
 <segment>
-<pinref part="SV1" gate="G$1" pin="6"/>
-<pinref part="SV1" gate="G$1" pin="5"/>
+<pinref part="FAN_C" gate="G$1" pin="6"/>
+<pinref part="FAN_C" gate="G$1" pin="5"/>
 <wire x1="449.58" y1="25.4" x2="464.82" y2="25.4" width="0.1524" layer="91"/>
 <wire x1="464.82" y1="25.4" x2="474.98" y2="25.4" width="0.1524" layer="91"/>
@@
 </segment>
 <segment>
-<pinref part="SV3" gate="G$1" pin="8"/>
-<pinref part="SV3" gate="G$1" pin="7"/>
+<pinref part="PREH_C" gate="G$1" pin="8"/>
+<pinref part="PREH_C" gate="G$1" pin="7"/>
 <wire x1="449.58" y1="52.07" x2="464.82" y2="52.07" width="0.1524" layer="91"/>
 <wire x1="464.82" y1="52.07" x2="473.71" y2="52.07" width="0.1524" layer="91"/>
@@
 </segment>
 <segment>
-<pinref part="SV1" gate="G$1" pin="10"/>
-<pinref part="SV1" gate="G$1" pin="9"/>
+<pinref part="FAN_C" gate="G$1" pin="10"/>
+<pinref part="FAN_C" gate="G$1" pin="9"/>
 <wire x1="449.58" y1="30.48" x2="464.82" y2="30.48" width="0.1524" layer="91"/>
 <wire x1="464.82" y1="30.48" x2="474.98" y2="30.48" width="0.1524" layer="91"/>
@@
 </segment>
 <segment>
-<pinref part="SV1" gate="G$1" pin="4"/>
-<pinref part="SV1" gate="G$1" pin="3"/>
+<pinref part="FAN_C" gate="G$1" pin="4"/>
+<pinref part="FAN_C" gate="G$1" pin="3"/>
 <wire x1="449.58" y1="22.86" x2="464.82" y2="22.86" width="0.1524" layer="91"/>
 <wire x1="464.82" y1="22.86" x2="474.98" y2="22.86" width="0.1524" layer="91"/>
@@
 </segment>
 <segment>
-<pinref part="SV3" gate="G$1" pin="4"/>
-<pinref part="SV3" gate="G$1" pin="3"/>
+<pinref part="PREH_C" gate="G$1" pin="4"/>
+<pinref part="PREH_C" gate="G$1" pin="3"/>
 <wire x1="449.58" y1="46.99" x2="464.82" y2="46.99" width="0.1524" layer="91"/>
 <wire x1="464.82" y1="46.99" x2="473.71" y2="46.99" width="0.1524" layer="91"/>
@@
 </segment>
 <segment>
-<pinref part="SV1" gate="G$1" pin="8"/>
-<pinref part="SV1" gate="G$1" pin="7"/>
+<pinref part="FAN_C" gate="G$1" pin="8"/>
+<pinref part="FAN_C" gate="G$1" pin="7"/>
 <wire x1="449.58" y1="27.94" x2="464.82" y2="27.94" width="0.1524" layer="91"/>
 <wire x1="464.82" y1="27.94" x2="474.98" y2="27.94" width="0.1524" layer="91"/>
@@
 </segment>
 <segment>
-<pinref part="SV3" gate="G$1" pin="6"/>
-<pinref part="SV3" gate="G$1" pin="5"/>
+<pinref part="PREH_C" gate="G$1" pin="6"/>
+<pinref part="PREH_C" gate="G$1" pin="5"/>
 <wire x1="449.58" y1="49.53" x2="464.82" y2="49.53" width="0.1524" layer="91"/>
 <wire x1="464.82" y1="49.53" x2="473.71" y2="49.53" width="0.1524" layer="91"/>
@@
 </segment>
 <segment>
-<pinref part="SV1" gate="G$1" pin="2"/>
-<pinref part="SV1" gate="G$1" pin="1"/>
+<pinref part="FAN_C" gate="G$1" pin="2"/>
+<pinref part="FAN_C" gate="G$1" pin="1"/>
 <wire x1="449.58" y1="20.32" x2="464.82" y2="20.32" width="0.1524" layer="91"/>
 <wire x1="464.82" y1="20.32" x2="474.98" y2="20.32" width="0.1524" layer="91"/>
@@
 </segment>
 <segment>
-<pinref part="SV3" gate="G$1" pin="2"/>
-<pinref part="SV3" gate="G$1" pin="1"/>
+<pinref part="PREH_C" gate="G$1" pin="2"/>
+<pinref part="PREH_C" gate="G$1" pin="1"/>
 <wire x1="449.58" y1="44.45" x2="464.82" y2="44.45" width="0.1524" layer="91"/>
 <wire x1="464.82" y1="44.45" x2="473.71" y2="44.45" width="0.1524" layer="91"/>

Commit message: .
Parts:
- added SV1: (no value), con-lstb:MA03-1
- 3D1: value IR2153P -> IR2153D; device DSS:IR2153P -> DSS:IR2153D
Connections:
- new net N$68: 1D4.O3, SV1.3
- net R_EXT: now also SV1.2
- net R_PREH: now also SV1.1
Other:
- moved on the sheet: 1C12, 1D3, 1D4, 1KK1, 1KK2, 1KK3, 1R30, 1R31, 1R32, 1VD1, 1VT1, 1X10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

Commit message: .
Parts:
- 3C10: device resistor:C-EU050-035X075 -> resistor:C-EU075-032X103
- 3R3: device resistor:R-EU_0613/5V -> resistor:R-EU_0613/15
- 3R5: device resistor:R-EU_M0805 -> resistor:R-EU_0207/7
- 3R6: device resistor:R-EU_M0805 -> resistor:R-EU_0207/10
- J1: value J5MM -> J7MM; device jumper:J5MM -> jumper:J7MM
Changed lines of the file:
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@@
 <attribute name="OC_NEWARK" value="29M3118"/>
 </part>
-<part name="3C10" library="resistor" deviceset="C-EU" device="050-035X075" value="470x2kv_K15-5"/>
+<part name="3C10" library="resistor" deviceset="C-EU" device="075-032X103" value="470x2kv_K15-5"/>
 <part name="3D2" library="v-reg" deviceset="78XXS" device="" value="7805"/>
 <part name="3C14" library="resistor" deviceset="CPOL-EU" device="E2.5-7" value="100x16v"/>
@@
 <part name="3VT1" library="transistor-power" deviceset="IRF740" device="" value="IRF740"/>
 <part name="3VT2" library="transistor-power" deviceset="IRF740" device="" value="IRF740"/>
-<part name="3R6" library="resistor" deviceset="R-EU_" device="M0805" value="27"/>
+<part name="3R6" library="resistor" deviceset="R-EU_" device="0207/10" value="27"/>
 <part name="3R4" library="resistor" deviceset="R-EU_" device="M0805" value="15k"/>
 <part name="3C6" library="resistor" deviceset="C-EU" device="050-025X075" value="1n"/>
@@
 <part name="3VD2" library="diode" deviceset="1N4004" device="" value="1N4007"/>
 <part name="3VDD3" library="diode" deviceset="1N4004" device="" value="1N4007"/>
-<part name="3R3" library="resistor" deviceset="R-EU_" device="0613/5V" value="36k 2w"/>
+<part name="3R3" library="resistor" deviceset="R-EU_" device="0613/15" value="36k 2w"/>
 <part name="3C5" library="rcl" deviceset="CPOL-EU" device="E3.5-8" value="100x25v"/>
 <part name="3C7" library="rcl" deviceset="CPOL-EU" device="E2.5-7" value="4.7x25v"/>
@@
 <part name="U$4" library="DSS" deviceset="R0.5W" device=""/>
 <part name="3D1" library="DSS" deviceset="IR2153" device="D" value="IR2153D"/>
-<part name="J1" library="jumper" deviceset="J" device="5MM"/>
+<part name="J1" library="jumper" deviceset="J" device="7MM" value="J7MM"/>
 <part name="MFRAME" library="DSS" deviceset="_SYMBOL" device="_MFRAME"/>
 <part name="PWO" library="con-wago-508" deviceset="W237-02P" device=""/>
@@
 <part name="4R14" library="resistor" deviceset="R-EU_" device="M0805" value="470"/>
 <part name="MFRAME_D" library="DSS" deviceset="_SYMBOL" device="_MFRAME"/>
-<part name="3R5" library="resistor" deviceset="R-EU_" device="M0805" value="27"/>
+<part name="3R5" library="resistor" deviceset="R-EU_" device="0207/7" value="27"/>
 <part name="4VD8" library="diode" deviceset="DIODE-" device="SOD80C"/>
 <part name="DISPL2" library="con-lstb" deviceset="MA03-2" device=""/>

Commit message: .
Parts:
- 3R4: device resistor:R-EU_M0805 -> resistor:R-EU_0204/7
Other:
- moved on the sheet: 1C17, 1OK1, 1R33, 1R36, 1R40, 1R43, 1T1, EXT-1, EXT-2
