File: DSS3P.sch (EAGLE design)
At the start: 290 parts, among them J1 J7MM

Commit message: a005
Parts:
- 1C9: device resistor:C-EUC0805 -> resistor:C-EUC1206
- 1R27: device resistor:R-EU_M0805 -> resistor:R-EU_R1206W
- AIR: value AIR -> (none)
- R_PW: value R_PW -> (none)
- renumbered 1X10 to AIR, 3SL2 to R_PW, PWFAN1 to PWPRH, SV1 to S_REL
Connections:
- net N$68 renamed R_FEN
- net ~220V_A: now also PWIE-2.KL; no longer PWIE-1.KL
- net ~220V_B: now also PWIE-1.KL; no longer PWIE-2.KL
Other:
- moved on the sheet: PWIE-1, PWIE-2

Commit message: a008
Connections:
- removed net N$47: 3C14.+, 3D2.OUT
- net +5V: now also 3C14.+, 3D2.OUT
Other:
- moved on the sheet: 1C1, 1C18, 1C19, 1C5, 1C8, 1D1A, 1OK2, 1OK3, 1R1, 1R13, 1R17, 1R22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

Commit message: .
Parts:
- added 2J6: 0, resistor:R-EU_R3225W
Connections:
- new net N$68: 2J6.1, DISPL1.5
- net +12V: no longer AIR.2, R_PW.2
- net +24V: now also AIR.2, R_PW.2
- net +5V: now also 2J6.2; no longer DISPL1.5
Other:
- moved on the sheet: 1C1, 1C17, 1C18, 1C19, 1C5, 1C8, 1D1A, 1OK1, 1OK2, 1OK3, 1R1, 1R13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

Commit message: ..
Parts:
- 1R33, 1R34, 1R35: device resistor:R-EU_M0805 -> resistor:R-EU_0207/10
Changed lines of the file:
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@@
 <setting verticaltext="up"/>
 </settings>
-<grid distance="100" unitdist="mil" unit="mil" style="lines" multiple="1" display="yes" altdistance="0.01" altunitdist="inch" altunit="inch"/>
+<grid distance="50" unitdist="mil" unit="mil" style="lines" multiple="1" display="yes" altdistance="0.01" altunitdist="inch" altunit="inch"/>
 <layers>
 <layer number="1" name="Top" color="4" fill="1" visible="yes" active="no"/>
@@
 <part name="1OK3" library="DSS" deviceset="MOC3063M" device="D" value="MOC3063"/>
 <part name="1T3" library="ON Semiconductor_simistor" deviceset="BTA16-600CW3G" device="TO220DS" value="BTA12-600CWRG"/>
-<part name="1R35" library="resistor" deviceset="R-EU_" device="M0805" value="510"/>
+<part name="1R35" library="resistor" deviceset="R-EU_" device="0207/10" value="510"/>
 <part name="1R42" library="resistor" deviceset="R-EU_" device="0207/10" value="390"/>
 <part name="1R39" library="resistor" deviceset="R-EU_" device="0613/15" value="390"/>
@@
 <part name="1OK1" library="DSS" deviceset="MOC3063M" device="D" value="MOC3063"/>
 <part name="1T1" library="ON Semiconductor_simistor" deviceset="BTA16-600CW3G" device="TO220DS" value="BTA12-600CWRG"/>
-<part name="1R33" library="resistor" deviceset="R-EU_" device="M0805" value="510"/>
+<part name="1R33" library="resistor" deviceset="R-EU_" device="0207/10" value="510"/>
 <part name="1R40" library="resistor" deviceset="R-EU_" device="0613/15" value="390"/>
 <part name="1R36" library="resistor" deviceset="R-EU_" device="0613/15" value="390"/>
@@
 <part name="1OK2" library="DSS" deviceset="MOC3063M" device="D" value="MOC3063"/>
 <part name="1T2" library="ON Semiconductor_simistor" deviceset="BTA16-600CW3G" device="TO220DS" value="BTA12-600CWRG"/>
-<part name="1R34" library="resistor" deviceset="R-EU_" device="M0805" value="510"/>
+<part name="1R34" library="resistor" deviceset="R-EU_" device="0207/10" value="510"/>
 <part name="1R41" library="resistor" deviceset="R-EU_" device="0613/15" value="390"/>
 <part name="1R37" library="resistor" deviceset="R-EU_" device="0613/15" value="390"/>
@@
 <text x="36.83" y="60.96" size="1.778" layer="94">1A</text>
 <text x="20.32" y="60.96" size="1.778" layer="94">6A</text>
-<wire x1="11.43" y1="285.75" x2="273.05" y2="285.75" width="0.4064" layer="90"/>
-<wire x1="273.05" y1="285.75" x2="273.05" y2="137.16" width="0.4064" layer="90"/>
+<wire x1="11.43" y1="284.48" x2="273.05" y2="284.48" width="0.4064" layer="90"/>
+<wire x1="273.05" y1="284.48" x2="273.05" y2="137.16" width="0.4064" layer="90"/>
 <wire x1="273.05" y1="137.16" x2="208.28" y2="137.16" width="0.4064" layer="90"/>
 <wire x1="208.28" y1="137.16" x2="208.28" y2="128.27" width="0.4064" layer="90"/>
@@
 <wire x1="53.34" y1="91.44" x2="53.34" y2="58.42" width="0.4064" layer="90"/>
 <wire x1="53.34" y1="58.42" x2="11.43" y2="58.42" width="0.4064" layer="90"/>
-<wire x1="11.43" y1="58.42" x2="11.43" y2="285.75" width="0.4064" layer="90"/>
+<wire x1="11.43" y1="58.42" x2="11.43" y2="284.48" width="0.4064" layer="90"/>
 <text x="292.1" y="73.66" size="1.778" layer="91">900
 3 H+
@@
 </instance>
 <instance part="U$2" gate="G$1" x="139.7" y="19.05"/>
-<instance part="GND1" gate="1" x="162.56" y="3.81" rot="MR0"/>
+<instance part="GND1" gate="1" x="162.56" y="5.08" rot="MR0"/>
 <instance part="S_REL" gate="G$1" x="589.28" y="162.56" smashed="yes" rot="MR0">
 <attribute name="VALUE" x="590.55" y="154.94" size="1.778" layer="96" rot="MR0"/>
@@
 <wire x1="160.02" y1="13.97" x2="162.56" y2="13.97" width="0.1524" layer="91"/>
 <pinref part="GND1" gate="1" pin="GND"/>
-<wire x1="162.56" y1="13.97" x2="162.56" y2="6.35" width="0.1524" layer="91"/>
+<wire x1="162.56" y1="13.97" x2="162.56" y2="7.62" width="0.1524" layer="91"/>
 </segment>
 </net>
@@
 <segment>
 <pinref part="4J4" gate="G$1" pin="2"/>
-<wire x1="110.49" y1="279.4" x2="113.03" y2="279.4" width="0.1524" layer="91"/>
-<label x="110.49" y="276.86" size="1.778" layer="95"/>
+<wire x1="110.49" y1="279.4" x2="116.84" y2="279.4" width="0.1524" layer="91"/>
+<label x="111.76" y="279.4" size="1.778" layer="95"/>
 </segment>
 <segment>
 <pinref part="4HL6" gate="G$1" pin="A"/>
 <wire x1="97.79" y1="250.19" x2="102.87" y2="250.19" width="0.1524" layer="91"/>
-<label x="100.33" y="250.19" size="1.778" layer="95"/>
+<label x="99.06" y="250.19" size="1.778" layer="95"/>
 </segment>
 </net>

Commit message: ..
Parts:
- 2J4: device resistor:R-EU_R3225W -> jumper:J7MM
Connections:
- net +5V: no longer 2D2P.VCC, 2R3.2, 2VD1.C, 2VD2.A
- net VCC: now also 2D2P.VCC, 2R3.2, 2VD1.C, 2VD2.A

Commit message: ..
Parts:
- 1R30, 1R31: device resistor:R-EU_M0805 -> resistor:R-EU_0207/10
Connections:
- net +5V: no longer 1R30.1
- net VCC: now also 1R30.1
