File: DSS3P.sch (EAGLE design)
At the start: 291 parts, among them J1 J7MM

Commit message: 2r7
Parts:
- added 2J7: 0, resistor:R-EU_R3225W
Connections:
- new net N$47: 2J7.2, AVR_ISP.7
- net TXD(RX): now also 2J7.1; no longer AVR_ISP.7
Other:
- moved on the sheet: 2J6, AIR, AVR_ISP, DISPL1

Commit message: r2
Connections:
- net N$159 renamed GND$159
- net N$80 renamed GND$80
Changed lines of the file:
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@@
 </segment>
 </net>
-<net name="N$159" class="0">
+<net name="GND$159" class="0">
 <segment>
 <pinref part="2D2" gate="P" pin="GND"/>
@@
 </segment>
 </net>
-<net name="N$80" class="0">
+<net name="GND$80" class="0">
 <segment>
 <wire x1="320.04" y1="233.68" x2="317.5" y2="233.68" width="0.1524" layer="91"/>

Commit message: usb fix
Connections:
- net N$17 renamed VCC_CH340G
- removed net N$157: 2D2B.A4, 2J2.2
- net TX: now also 2D2B.A4; no longer 2J2.1
Other:
- moved on the sheet: 2J2
Changed lines of the file:
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@@
 <attribute name="VALUE" x="284.48" y="184.658" size="1.778" layer="96"/>
 </instance>
-<instance part="2J2" gate="G$1" x="358.14" y="203.2" smashed="yes">
-<attribute name="NAME" x="354.33" y="199.6186" size="1.778" layer="95"/>
-<attribute name="VALUE" x="364.49" y="201.422" size="1.778" layer="96" rot="R180"/>
+<instance part="2J2" gate="G$1" x="358.14" y="175.26" smashed="yes">
+<attribute name="NAME" x="354.33" y="171.6786" size="1.778" layer="95"/>
+<attribute name="VALUE" x="364.49" y="173.482" size="1.778" layer="96" rot="R180"/>
 </instance>
 <instance part="2VT1" gate="G$1" x="299.72" y="185.42" smashed="yes" rot="MR0">
@@
 </segment>
 </net>
-<net name="N$17" class="0">
+<net name="VCC_CH340G" class="0">
 <segment>
 <wire x1="347.98" y1="210.82" x2="347.98" y2="218.44" width="0.1524" layer="91"/>
@@
 </segment>
 <segment>
-<label x="347.98" y="203.2" size="1.778" layer="95"/>
-<wire x1="347.98" y1="203.2" x2="353.06" y2="203.2" width="0.1524" layer="91"/>
-<pinref part="2J2" gate="G$1" pin="1"/>
+<label x="355.6" y="203.2" size="1.778" layer="95"/>
+<wire x1="355.6" y1="203.2" x2="368.3" y2="203.2" width="0.1524" layer="91"/>
+<pinref part="2D2" gate="B" pin="A4"/>
 </segment>
 <segment>
@@
 </segment>
 </net>
-<net name="N$157" class="0">
-<segment>
-<pinref part="2J2" gate="G$1" pin="2"/>
-<pinref part="2D2" gate="B" pin="A4"/>
-<wire x1="363.22" y1="203.2" x2="368.3" y2="203.2" width="0.1524" layer="91"/>
-</segment>
-</net>

Commit message: gnd+1
Parts:
- removed VD2: 1N4148DO35-7, diode:1N4148DO35-7
- added 2VD3: LL4148, diode:DIODE-SOD80C
- added VD1: 1N4148DO35-7, diode:1N4148DO35-7
Connections:
- net VCC: now also 2VD3.C; no longer VD2.C
- net V_PROG: now also 2VD3.A; no longer VD2.A
Changed lines of the file:
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@@
 <part name="1R32" library="resistor" deviceset="R-EU_" device="M0805" value="10k"/>
 <part name="1VD1" library="diode" deviceset="1N4148" device="DO35-7"/>
-<part name="VD2" library="diode" deviceset="1N4148" device="DO35-7"/>
 <part name="1R30" library="resistor" deviceset="R-EU_" device="0207/10" value="10k"/>
 <part name="1D1" library="linear" deviceset="LM358" device="D" value="LM358D"/>
@@
 <part name="P+20" library="supply1" deviceset="VCC" device=""/>
 <part name="2J7" library="resistor" deviceset="R-EU_" device="R3225W" value="0"/>
+<part name="VD1" library="diode" deviceset="1N4148" device="DO35-7"/>
+<part name="2VD3" library="diode" deviceset="DIODE-" device="SOD80C" value="LL4148"/>
 </parts>
 <sheets>
@@
 <attribute name="NAME" x="418.5666" y="166.37" size="1.778" layer="95" rot="R270"/>
 </instance>
-<instance part="VD2" gate="G$1" x="424.18" y="185.42" smashed="yes" rot="R270">
-<attribute name="NAME" x="427.2534" y="177.8" size="1.778" layer="95" rot="R90"/>
-</instance>
 <instance part="1R30" gate="G$1" x="539.75" y="210.82" smashed="yes" rot="R270">
 <attribute name="NAME" x="532.13" y="208.5086" size="1.778" layer="95"/>
@@
 <attribute name="NAME" x="509.0414" y="209.55" size="1.778" layer="95" rot="R90"/>
 <attribute name="VALUE" x="507.238" y="219.71" size="1.778" layer="96" rot="R270"/>
+</instance>
+<instance part="VD1" gate="G$1" x="378.46" y="175.26" smashed="yes" rot="R270">
+<attribute name="NAME" x="381.5334" y="167.64" size="1.778" layer="95" rot="R90"/>
+</instance>
+<instance part="2VD3" gate="G$1" x="424.18" y="185.42" smashed="yes" rot="MR270">
+<attribute name="NAME" x="419.5826" y="182.88" size="1.778" layer="95" rot="MR90"/>
+<attribute name="VALUE" x="416.7886" y="180.34" size="1.778" layer="96" rot="MR90"/>
 </instance>
 </instances>
@@
 <pinref part="1VD1" gate="G$1" pin="C"/>
 <pinref part="1D3" gate="1" pin="VCC@1"/>
-<pinref part="VD2" gate="G$1" pin="C"/>
 <wire x1="424.18" y1="182.88" x2="424.18" y2="162.56" width="0.1524" layer="91"/>
 <junction x="424.18" y="162.56"/>
@@
 <pinref part="P+19" gate="VCC" pin="VCC"/>
 <wire x1="416.56" y1="162.56" x2="421.64" y2="162.56" width="0.1524" layer="91"/>
+<pinref part="2VD3" gate="G$1" pin="C"/>
 </segment>
 <segment>
@@
 <segment>
 <label x="423.672" y="198.12" size="1.778" layer="95" rot="R90"/>
-<pinref part="VD2" gate="G$1" pin="A"/>
 <wire x1="424.18" y1="187.96" x2="424.18" y2="210.82" width="0.1524" layer="91"/>
 <wire x1="424.18" y1="210.82" x2="482.6" y2="210.82" width="0.1524" layer="91"/>
@@
 <pinref part="AVR_ISP" gate="G$1" pin="2"/>
 <wire x1="482.6" y1="238.76" x2="495.3" y2="238.76" width="0.1524" layer="91"/>
-</segment>
-</net>
+<pinref part="2VD3" gate="G$1" pin="A"/>
+</segment>
+</net>

Commit message: .
Changed lines of the file:
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@@
-</segment>
-</net>
-<net name="N$125" class="0">
-<segment>
-<pinref part="4VT1" gate="G$1" pin="C"/>
-<wire x1="589.28" y1="210.82" x2="589.28" y2="212.09" width="0.1524" layer="91"/>
-<label x="588.01" y="212.09" size="1.778" layer="95" rot="R180"/>
 </segment>
 </net>
@@
 <junction x="327.66" y="193.04"/>
 <label x="330.2" y="185.42" size="1.778" layer="95"/>
-<wire x1="327.66" y1="185.42" x2="337.82" y2="185.42" width="0.1524" layer="91"/>
+<wire x1="327.66" y1="185.42" x2="340.36" y2="185.42" width="0.1524" layer="91"/>
 <junction x="327.66" y="185.42"/>
 </segment>
@@
 </segment>
 </net>
+<net name="N$17" class="0">
+<segment>
+<pinref part="4VT1" gate="G$1" pin="C"/>
+<wire x1="589.28" y1="210.82" x2="589.28" y2="213.36" width="0.1524" layer="91"/>
+<wire x1="589.28" y1="213.36" x2="584.2" y2="213.36" width="0.1524" layer="91"/>
+</segment>
+</net>

Commit message: +pow
Parts:
- renumbered 2VD3 to 1VD3
Changed lines of the file:
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@@
 <?xml version="1.0" encoding="utf-8"?>
 <!DOCTYPE eagle SYSTEM "eagle.dtd">
-<eagle version="6.4">
+<eagle version="6.3">
 <drawing>
 <settings>
@@
 <part name="2J7" library="resistor" deviceset="R-EU_" device="R3225W" value="0"/>
 <part name="VD1" library="diode" deviceset="1N4148" device="DO35-7"/>
-<part name="2VD3" library="diode" deviceset="DIODE-" device="SOD80C" value="LL4148"/>
+<part name="1VD3" library="diode" deviceset="DIODE-" device="SOD80C" value="LL4148"/>
 </parts>
 <sheets>
@@
 <attribute name="NAME" x="381.5334" y="167.64" size="1.778" layer="95" rot="R90"/>
 </instance>
-<instance part="2VD3" gate="G$1" x="424.18" y="185.42" smashed="yes" rot="MR270">
+<instance part="1VD3" gate="G$1" x="424.18" y="185.42" smashed="yes" rot="MR270">
 <attribute name="NAME" x="419.5826" y="182.88" size="1.778" layer="95" rot="MR90"/>
 <attribute name="VALUE" x="416.7886" y="180.34" size="1.778" layer="96" rot="MR90"/>
@@
 <pinref part="P+19" gate="VCC" pin="VCC"/>
 <wire x1="416.56" y1="162.56" x2="421.64" y2="162.56" width="0.1524" layer="91"/>
-<pinref part="2VD3" gate="G$1" pin="C"/>
+<pinref part="1VD3" gate="G$1" pin="C"/>
 </segment>
 <segment>
@@
 <pinref part="AVR_ISP" gate="G$1" pin="2"/>
 <wire x1="482.6" y1="238.76" x2="495.3" y2="238.76" width="0.1524" layer="91"/>
-<pinref part="2VD3" gate="G$1" pin="A"/>
+<pinref part="1VD3" gate="G$1" pin="A"/>
 </segment>
 </net>
