File: DSS3P.brd (EAGLE design)
At the start: 399.7 x 251.8 mm, 299 parts, among them J1 J7MM

Commit message: +epf
Parts:
- moved 1VT1 0.32 mm to (127.3, 152.7)
Changed lines of the file:
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@@
 </element>
 <element name="1R31" library="resistor" package="0207/10" value="33k" x="136.525" y="132.715" rot="R270"/>
-<element name="1VT1" library="transistor" package="TO92-ECB" value="" x="127.3175" y="153.035" rot="R270"/>
+<element name="1VT1" library="transistor" package="TO92-ECB" value="" x="127.3175" y="152.7175" rot="R270"/>
 <element name="SG1" library="buzzer" package="F/CM12P" value="F/CM12P" x="117.7925" y="153.035" rot="R180">
 <attribute name="OC_NEWARK" value="unknown" x="-47.307496875" y="215.265003125" size="1.778" layer="27" rot="R180" display="off"/>
@@
 <wire x1="152.7175" y1="137.795" x2="154.94" y2="137.795" width="1.27" layer="16"/>
 <wire x1="154.94" y1="125.73" x2="153.3525" y2="124.46" width="1.27" layer="16"/>
-<wire x1="127.3175" y1="155.575" x2="127.3175" y2="158.115" width="0.6096" layer="16"/>
+<wire x1="127.3175" y1="155.2575" x2="127.3175" y2="158.115" width="0.6096" layer="16"/>
 <wire x1="127.3175" y1="158.115" x2="128.905" y2="159.7025" width="0.6096" layer="16"/>
 <wire x1="128.905" y1="159.7025" x2="133.985" y2="159.7025" width="0.6096" layer="16"/>
@@
 <contactref element="1VT1" pad="B"/>
 <contactref element="1R32" pad="1"/>
-<wire x1="126.0475" y1="147.9525" x2="127.3175" y2="150.495" width="0.6096" layer="16"/>
+<wire x1="126.0475" y1="147.9525" x2="127.3175" y2="150.1775" width="0.6096" layer="16"/>
 </signal>
 <signal name="V_PROG">
@@
 <contactref element="1VT1" pad="C"/>
 <contactref element="SG1" pad="-"/>
-<wire x1="121.6025" y1="153.035" x2="127.3175" y2="153.035" width="0.6096" layer="16"/>
+<wire x1="121.6025" y1="153.035" x2="127.3175" y2="152.7175" width="0.6096" layer="16"/>
 </signal>
 <signal name="N$14">

Commit message: 11
Parts:
- moved 2VD2 4.80 mm to (139.1, 174.9)
- moved 1VD1 1.31 mm to (133.0, 168.6)
- moved 1VT1 0.32 mm to (127.3, 153.0)
Routing:
- net VCC: track 156.6 -> 161.4 mm
- net VCC_CH340G: track 15.1 -> 16.6 mm
- net +5V: track 282.1 -> 283.4 mm
- net USB_SEL: track 69.5 -> 70.4 mm
- net GND: track 797.6 -> 797.0 mm

Commit message: .
Parts:
- moved 2R6 12.4 mm to (153.4, 147.0)
- moved 2R4 1.14 mm to (154.3, 166.1)
Routing:
- net USB_SEL: track 70.4 -> 74.3 mm
- net N$176: track 3.06 -> 2.44 mm

Commit message: .t
Parts:
- 1D4: value ULN2003D -> ULN2003N
- 1VT1: value (none) -> КТ315Б
- 3C11: device DSS:C_D25-12 -> DSS0:C_D25-12
- 3C3, 3C4: device DSS:C_22X10 -> DSS0:C_22X10
- 4VT1: value BC547 -> КТ315Б; device transistor-neu-to92:TO92 -> transistor:TO92-ECB
- moved S2_S 30.5 mm to (153.0, 54.9)
- moved 4VT1 23.8 mm to (153.0, 57.1), turned to 0 degrees
- moved 4C4 15.6 mm to (153.4, 61.3)
- moved 4R12 9.71 mm to (153.4, 64.1), turned to 180 degrees
- moved 4VD13 6.74 mm to (148.9, 64.1), turned to 0 degrees
- moved 1R22A 0.95 mm to (147.0, 87.8)
- moved 1C8 0.71 mm to (141.6, 91.1)
- moved 1R12 0.32 mm to (115.1, 76.2)
- moved 1R15 0.32 mm to (104.9, 79.2)
- moved 1VD3 0.32 mm to (151.1, 130.2)
- moved 2J6 0.32 mm to (148.0, 120.0)
- moved 2R2 0.32 mm to (135.3, 203.4)
- flipped 1R1 to the top
- flipped 1R17 to the top
- flipped 1R18 to the top
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Connections:
- net GND: now also 4VT1.E; no longer 4VT1.1
- net N$127: now also 4VT1.B; no longer 4VT1.2
- net N$17: now also 4VT1.C; no longer 4VT1.3
Routing:
- net N$165: track 53.9 -> 82.1 mm
- net TI_PREHEAT: track 59.3 -> 38.1 mm
- net POWER+: track 62.7 -> 52.7 mm
- net PWM_SOL_2: track 85.1 -> 75.8 mm
- net GND: track 797.4 -> 800.8 mm
- net M_PRH: track 66.5 -> 68.3 mm
- net T_PREHEAT: track 62.1 -> 63.3 mm
- net N$17: track 3.17 -> 2.22 mm
- net ~220V_A: track 104.0 -> 104.9 mm
- net N$128: track 2.64 -> 1.80 mm
- net BUZZER: track 35.5 -> 36.3 mm
- net N$24: track 12.4 -> 11.7 mm
- net PWM_SOL_1: track 79.4 -> 80.1 mm
- net TXD(RX): track 97.1 -> 97.7 mm
- net VCC_CH340G: track 16.6 -> 16.0 mm
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Other:
- board text added: "1170-18"

Commit message: topsilk
Parts:
- 3VD1: device DSS:ZDMETAL -> DSS0:ZDMETAL
- moved 3VD1 0.32 mm to (76.8, 125.7)

Commit message: l
Parts:
- 2C3, 2C4, 2C5: value (none) -> x
- moved 1SJ9 0.32 mm to (105.1, 51.4)
- moved 1VD2 0.32 mm to (116.4, 69.8)

Commit message: lab bot
Parts:
- moved 1R16 0.63 mm to (123.0, 83.5)
