File: DSS3P.brd (EAGLE design)
At the start: 399.7 x 251.8 mm, 330 parts, among them J1 J12MM, T1 E33

Commit message: f4
Parts:
- added 1VT1B1: BC847, transistor:SOT23
- added B2: BUZZER, DSS0:BUZZER
- moved 1C12 0.71 mm to (131.1, 127.6)
- moved 1D3 0.71 mm to (130.2, 120.5)
- moved 1R30 0.71 mm to (127.0, 127.3)
- moved U$12 0.71 mm to (122.6, 120.5)
- moved U$8 0.71 mm to (140.6, 120.5)
- moved U$13 0.71 mm to (131.6, 111.5)
- moved U$9 0.71 mm to (131.6, 129.5)
Connections:
- new net N$5: 1VT1B1.3, B2.-
- net GND: now also 1VT1B1.2
Routing:
- net BUZZER: track 50.5 -> 54.3 mm
- net KEY(SCK): track 124.0 -> 121.7 mm
- net T_PREHEAT: track 73.0 -> 74.9 mm
- net PWM_SOL_2: track 85.1 -> 83.3 mm
- net PWM_PRH(MISO): track 168.6 -> 167.1 mm
- net GND: track 848.8 -> 850.1 mm
- net TO_FAN: track 59.4 -> 58.1 mm
- net TXD(RX): track 87.5 -> 88.5 mm
- net PWM_FEN_P: track 97.7 -> 98.3 mm
- net VCC: track 180.2 -> 180.9 mm
- net GERKON: track 120.3 -> 119.7 mm

Commit message: sav
Parts:
- removed 1R32: 10k, resistor:M0805
- removed 1VT1: KT315, transistor:TO92-ECB
- removed 1VT1B, 1VT1B1: BC847, transistor:SOT23
- removed B1: BUZZER, DSS0:BUZZER
- added 1R47: 10k, resistor:M0805
- added 1VT7: KT315, transistor:TO92-ECB
- moved 1R31 29.6 mm to (153.4, 153.4), turned to 0 degrees
- moved 2J6 8.32 mm to (156.4, 115.9), turned to 270 degrees
- moved 1VD3 5.12 mm to (155.6, 132.7), turned to 0 degrees
- moved DISPL1 4.97 mm to (152.4, 120.7)
- moved B2 3.62 mm to (124.5, 104.1), turned to 225 degrees
- renumbered LED2 to LED
Connections:
- removed net BZB: 1R32.1, 1VT1.B, 1VT1B.1
- removed net BZK: 1VT1.C, 1VT1B.3, B1.-
- new net N$7: 1R47.1, 1VT7.B
- net +5V: now also B2.+; no longer B1.+
- net BUZZER: now also 1R47.2; no longer 1R32.2
- net GND: now also 1VT7.E; no longer 1VT1.E, 1VT1B.2, 1VT1B1.2
- net N$5: now also 1VT7.C; no longer 1VT1B1.3
Routing:
- net BUZZER: track 54.3 -> 6.81 mm, vias 2 -> 0
- net RXD(TX): track 95.0 -> 116.3 mm
- net T_SOLDER_2: track 51.8 -> 70.7 mm
- net T_SOLDER_1: track 55.5 -> 73.2 mm, vias 0 -> 2
- net +5V: track 292.3 -> 307.9 mm, vias 7 -> 9
- net BZK: track 14.6 -> 0.00 mm
- net RESET: track 80.4 -> 94.8 mm
- net STROB: track 6.83 -> 19.4 mm
- net GND: track 850.1 -> 862.3 mm
- net CLK: track 10.9 -> 22.0 mm
- net VCC: track 180.9 -> 171.0 mm
- net PWM_PRH(MISO): track 167.1 -> 175.8 mm
- net BZB: track 8.52 -> 0.00 mm
- net PD3: track 29.6 -> 36.4 mm
- net T_PREHEAT: track 74.9 -> 81.1 mm
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
Commit message: temp1
Parts:
- moved S_REL 30.4 mm to (118.1, 143.5), turned to 0 degrees
- moved R_PW 29.0 mm to (132.1, 143.8), turned to 0 degrees
- moved AIR 27.4 mm to (126.0, 143.8), turned to 180 degrees
- moved 1VT7 21.1 mm to (115.6, 121.0), turned to 270 degrees
- moved 1R47 20.8 mm to (117.8, 116.8), turned to 180 degrees
- moved B2 19.1 mm to (110.8, 117.5), turned to 270 degrees
- moved 1D4 18.5 mm to (123.2, 136.0), turned to 0 degrees
- moved U$13 14.1 mm to (121.0, 120.9), turned to 90 degrees
- moved U$8 13.6 mm to (130.0, 111.9), turned to 180 degrees
- moved U$12 12.0 mm to (130.0, 129.9), turned to 0 degrees
- moved U$9 11.4 mm to (139.0, 120.9), turned to 270 degrees
- moved 1R30 10.0 mm to (136.8, 125.4), turned to 90 degrees
- moved 1C12 8.76 mm to (137.2, 121.3), turned to 270 degrees
- moved 1D3 1.75 mm to (130.0, 122.2), turned to 180 degrees
- moved 1R31 0.32 mm to (153.0, 153.4)
Routing:
- net PWM_SOL_1: track 98.4 -> 48.6 mm
- net T_PREHEAT: track 81.1 -> 37.2 mm, vias 0 -> 2
- net M_PRH: track 64.4 -> 103.4 mm
- net T_SOLDER_2: track 70.7 -> 33.3 mm, vias 0 -> 2
- net TO_FAN: track 56.6 -> 23.1 mm, vias 2 -> 1
- net TXD(RX): track 86.5 -> 54.8 mm, vias 2 -> 0
- net M_FEN: track 71.8 -> 96.5 mm
- net +5V: track 307.9 -> 283.7 mm
- net GERKON: track 120.0 -> 101.1 mm, vias 2 -> 3
- net RXD(TX): track 116.3 -> 131.9 mm, vias 4 -> 6
- net T_SOLDER_1: track 73.2 -> 58.3 mm
- net KEY(SCK): track 120.0 -> 105.7 mm, vias 4 -> 0
- net CLK: track 22.0 -> 36.0 mm
- net VCC: track 171.0 -> 158.0 mm, vias 2 -> 4
- net ~220V_B: track 98.7 -> 111.6 mm
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
Commit message: test2
Parts:
- added 1C13: 100n, resistor:C0805
- 1R35: device resistor:0207/10 -> resistor:0207/15
- moved B2 9.84 mm to (109.1, 127.2), turned to 180 degrees
- moved PREH_C 5.12 mm to (152.7, 102.2)
- moved 1VT7 4.15 mm to (112.7, 118.0)
- moved 1R47 3.71 mm to (115.3, 114.1)
- moved 1VD3 2.25 mm to (155.3, 130.5), turned to 90 degrees
- moved 3C15 1.62 mm to (94.3, 106.0)
- moved 1R35 1.59 mm to (90.8, 72.1)
- moved 1D4 1.59 mm to (123.2, 137.6)
- moved S_REL 1.31 mm to (116.8, 143.8)
- moved R_PW 1.28 mm to (130.8, 144.0)
- moved 1D3 0.90 mm to (129.4, 121.6)
- moved U$12 0.90 mm to (129.4, 129.2)
- moved U$8 0.90 mm to (129.4, 111.2)
- moved U$13 0.90 mm to (120.4, 120.2)
- moved U$9 0.90 mm to (138.4, 120.2)
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Connections:
- net +24V: now also AIR.1; no longer AIR.2
- net GND: now also 1C13.2
- net M_AIR: now also AIR.2; no longer AIR.1
- net VCC: now also 1C13.1
Routing:
- net PWM_SOL_1: track 48.6 -> 146.5 mm, vias 0 -> 2
- net TXD(RX): track 54.8 -> 115.4 mm, vias 0 -> 2
- net TO_FAN: track 23.1 -> 71.3 mm, vias 1 -> 5
- net M_PRH: track 103.4 -> 123.3 mm
- net M_FEN: track 96.5 -> 111.4 mm
- net GND: track 859.2 -> 848.3 mm, vias 8 -> 10
- net N$5: track 4.77 -> 13.1 mm
- net PWM_FEN_P: track 105.3 -> 109.9 mm, vias 2 -> 0
- net TI_PREHEAT: track 37.5 -> 41.4 mm
- net PD3: track 39.8 -> 43.2 mm
- net RELAY_EXT: track 13.0 -> 16.0 mm
- net RELAY_FEN: track 10.3 -> 13.1 mm
- net +5V: track 283.7 -> 281.0 mm
- net PWM_EXT: track 187.0 -> 189.6 mm
- net T_SOLDER_1: track 58.3 -> 60.7 mm
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
Commit message: .
Routing:
- net GERKON: track 103.2 -> 100.1 mm, vias 4 -> 2
- net +5V: track 281.0 -> 278.6 mm
- net DATA: track 31.7 -> 32.8 mm
- net RXD(TX): track 130.8 -> 131.8 mm
- net STROB: track 31.1 -> 32.0 mm
- net PWM_PRH(MISO): track 164.0 -> 163.2 mm
- net T_SOLDER_1: track 60.7 -> 61.5 mm, vias 2 -> 4
- net CLK: track 35.5 -> 36.1 mm
- net KEY(SCK): track 106.6 -> 106.0 mm
- net PWM_SOL_2: vias 2 -> 0

Commit message: .
Routing:
- net M_PRH: track 123.3 -> 127.7 mm
- net PWM_PRH(MISO): track 163.2 -> 165.4 mm
- net PWM_SOL_2: track 80.0 -> 82.3 mm
- net +24V: track 265.9 -> 264.1 mm
- net RXD(TX): track 131.8 -> 133.4 mm
- net T_SOLDER_2: track 32.9 -> 31.4 mm
- net RESET: track 106.0 -> 104.6 mm
- net KEY(SCK): track 106.0 -> 104.7 mm
- net TO_FAN: track 71.2 -> 72.4 mm
- net T_PREHEAT: track 36.3 -> 35.3 mm
- net TXD(RX): track 114.9 -> 115.6 mm, vias 2 -> 4
- net N$165: track 81.3 -> 80.7 mm
- net GND: track 848.3 -> 848.9 mm
- net TI_PREHEAT: track 41.4 -> 42.0 mm
- added copper zone on layer 16, net GND
- added copper zone on layer 16, net GNS1
- added copper zone on layer 16, net GNS2

Commit message: .
Parts:
- moved DISPL1 6.35 mm to (152.2, 114.3)
- moved 2J6 1.60 mm to (156.2, 114.3)
- moved S_REL 1.50 mm to (118.1, 144.6)
- moved AIR 1.42 mm to (124.5, 144.6)
- moved R_PW 1.42 mm to (129.5, 144.6)
- moved 1R33 1.14 mm to (91.4, 96.2)
- moved PREH_C 1.00 mm to (153.7, 101.9), turned to 270 degrees
Routing:
- net N$68: track 9.93 -> 3.13 mm
- net DATA: track 32.3 -> 27.2 mm
- net PWM_PRH(MISO): track 165.4 -> 160.6 mm
- net TI_PREHEAT: track 42.0 -> 37.3 mm
- net STROB: track 32.0 -> 27.9 mm
- net +24V: track 264.1 -> 267.9 mm
- net TXD(RX): track 115.6 -> 119.5 mm
- net TO_FAN: track 72.4 -> 68.8 mm
- net KEY(SCK): track 104.7 -> 101.8 mm
- net T_SOLDER_2: track 31.4 -> 34.3 mm
- net M_PRH: track 127.7 -> 124.8 mm
- net GERKON: track 100.1 -> 97.6 mm
- net GND: track 848.9 -> 846.5 mm, vias 10 -> 8
- net CLK: track 36.1 -> 34.1 mm
- net T_SOLDER_1: track 61.3 -> 62.7 mm
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
Commit message: .
Parts:
- 1R31: device resistor:0207/10 -> resistor:M0805
- moved 1R31 34.4 mm to (146.1, 119.7), flipped to the bottom, turned to 90 degrees
- moved 1VD3 2.56 mm to (156.5, 132.7), turned to 0 degrees
Routing:
- net KEY(SCK): track 101.8 -> 126.9 mm
- net PWM_PRH(MISO): track 160.6 -> 174.3 mm, vias 1 -> 2
- net VCC: track 159.0 -> 164.9 mm
- net +5V: track 278.7 -> 280.6 mm
- net RXD(TX): track 133.5 -> 131.7 mm
- net T_SOLDER_2: track 34.3 -> 36.0 mm
- net T_SOLDER_1: track 62.7 -> 64.3 mm
- net PWM_SOL_2: track 82.5 -> 83.7 mm
- net RESET: track 104.9 -> 105.9 mm
- net TXD(RX): track 119.5 -> 120.2 mm, vias 4 -> 2
