File: DSS3P.brd (EAGLE design)
At the start: 399.7 x 251.8 mm, 333 parts, among them J1 J12MM, T1 E33

Commit message: .
Parts:
- moved 1R47 0.57 mm to (125.6, 110.0)
Routing:
- net GND: track 856.1 -> 849.4 mm
- net +24V: track 267.6 -> 268.7 mm
- net GERKON: track 110.1 -> 109.4 mm
- net BUZZER: track 9.25 -> 9.76 mm
- net N$7: track 9.88 -> 9.36 mm

Commit message: ..
Parts:
- moved 3VD10 1.60 mm to (80.3, 120.2)
- moved 3C15 1.42 mm to (92.1, 104.8)
- moved 3VD1 0.95 mm to (75.6, 124.5)
Routing:
- net GND: track 849.4 -> 846.9 mm
- net POWER-T: track 180.4 -> 178.4 mm
- net IRD: track 13.0 -> 14.8 mm
- net IRVCC: track 68.9 -> 70.1 mm
- net IRCT: track 22.1 -> 21.0 mm
- net M_PRH: track 96.1 -> 95.1 mm
- net PWM_PRH(MISO): track 176.7 -> 175.8 mm

Commit message: 7
Parts:
- moved 1R31 41.0 mm to (150.7, 113.3), turned to 90 degrees
- moved DISPL1 1.59 mm to (154.5, 114.3)
- moved PREH_C 0.79 mm to (154.5, 101.9)
Routing:
- net KEY(SCK): track 115.7 -> 121.0 mm
- net VCC: track 176.7 -> 181.1 mm
- net RESET: track 104.2 -> 106.5 mm
- net CLK: track 28.7 -> 30.4 mm
- net STROB: track 25.5 -> 27.1 mm
- net DATA: track 25.9 -> 27.5 mm
- net GND: track 846.9 -> 845.7 mm
- net PWM_PRH(MISO): track 175.8 -> 174.6 mm
- net M_PRH: track 95.1 -> 95.8 mm
- net +24V: track 268.7 -> 269.5 mm
- net TI_PREHEAT: track 35.1 -> 35.8 mm

Commit message: .
Parts:
- added DISPL3, DISPL4: (no value), con-lstb:MA03-2
- moved 2R5 9.69 mm to (140.8, 170.2)
- moved 2J7 3.50 mm to (146.1, 143.0)
- moved 2R6 1.46 mm to (153.7, 145.6)
- moved PREH_C 0.95 mm to (154.5, 102.9)
- moved 2R4 0.48 mm to (154.3, 165.6)
- moved 2VT1 0.48 mm to (155.3, 169.1)
- moved 2C5 0.35 mm to (138.4, 178.6)
- moved 3VD7 0.16 mm to (114.0, 176.1)
Routing:
- net +24V: track 269.5 -> 280.9 mm
- net N$47: track 7.27 -> 3.77 mm
- net POWER: track 0.00 -> 3.33 mm
- net R_PREH: track 0.00 -> 3.33 mm
- net R_EXT: track 0.00 -> 3.33 mm
- net R_FEN: track 0.00 -> 3.33 mm
- net M_AIR: track 0.00 -> 3.33 mm
- net USB_SEL: track 49.3 -> 50.7 mm
- net T_PREHEAT: track 53.4 -> 52.0 mm
- net RESET: track 106.5 -> 105.2 mm
- net TXD(RX): track 111.1 -> 110.0 mm
- net PWM_EXT: track 173.6 -> 174.6 mm
- net KEY(SCK): track 121.0 -> 122.0 mm
- net VCC: track 181.1 -> 180.4 mm
- net GND: track 845.7 -> 845.0 mm
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
Commit message: .
Parts:
- removed 3R8: 1e5* 2w, resistor:P0613/15
- added 1C14: (no value), resistor:C0805
- added R1, R2, R3, R4, R5, R6: (no value), rcl:R2010
- 2J7: device resistor:R3225W -> resistor:R1206W
- moved 3VD11 8.53 mm to (77.0, 177.0), turned to 0 degrees
- moved 3R7 3.03 mm to (68.1, 189.5)
- moved 3C10 0.79 mm to (103.5, 163.4), turned to 30 degrees
- moved 3C14 0.79 mm to (114.5, 162.2), turned to 180 degrees
- moved 1R47 0.63 mm to (126.2, 110.0)
- moved 3VD12 0.45 mm to (72.4, 170.5), turned to 270 degrees
- moved 2VD2 0.16 mm to (136.7, 174.6)
Connections:
- new net N$8: R1.1, R2.1, R3.1, R4.2, R5.2, R6.2
- net GND: now also 1C14.2
- net N$7: now also 1C14.1
- net POWER-: now also R1.2, R2.2, R3.2; no longer 3R8.2
- net POWER-T: now also R4.1, R5.1, R6.1; no longer 3R8.1
Routing:
- net N$4: track 0.00 -> 27.5 mm
- net POWER-: track 103.8 -> 125.1 mm
- net N$8: track 0.00 -> 20.8 mm
- net POWER+: track 57.6 -> 46.6 mm
- net GND: track 845.0 -> 855.6 mm
- net N$1: track 0.00 -> 4.40 mm
- net N$3: track 0.00 -> 4.25 mm
- net DD: track 106.8 -> 103.2 mm
- net M_FEN: track 84.2 -> 82.0 mm
- net POWER-T: track 178.4 -> 176.4 mm
- net PWM_PRH(MISO): track 174.7 -> 172.8 mm
- net +5V: track 240.9 -> 240.2 mm, vias 8 -> 9
- net N$99: track 9.72 -> 10.5 mm
- net N$98: track 11.9 -> 12.5 mm
- net KEY(SCK): track 122.0 -> 121.3 mm
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
Commit message: .
Parts:
- moved DISPL3 74.5 mm to (127.3, 149.2), turned to 45 degrees
- moved R_PW 2.25 mm to (117.0, 139.4), turned to 225 degrees
- moved AIR 2.02 mm to (113.2, 135.6), turned to 225 degrees
- moved 3C6 1.91 mm to (84.9, 129.5)
Connections:
- net +24V: now also R_PW.1; no longer R_PW.2
- net POWER: now also R_PW.2; no longer R_PW.1
Routing:
- net M_FEN: track 82.0 -> 94.3 mm
- net M_PRH: track 96.2 -> 108.2 mm
- net IRVCC: track 70.1 -> 74.1 mm
- net M_AIR: track 3.33 -> 0.00 mm
- net PWM_PRH(MISO): track 172.8 -> 170.9 mm
- net +24V: track 280.9 -> 282.7 mm
- net +5V: track 240.2 -> 241.8 mm
- net IRCT: track 21.0 -> 22.7 mm
- net GND: track 855.6 -> 857.1 mm
- net PWM_EXT: track 174.3 -> 172.9 mm
- net PWM_FEN_P: track 90.9 -> 90.0 mm
- net POWER: track 3.33 -> 4.07 mm
- net POWER-T: track 176.4 -> 177.0 mm

Commit message: .
Parts:
- removed AIR, R_PW: (no value), con-amp-quick:02P
- removed DISPL3, DISPL4: (no value), con-lstb:MA03-2
- added AIR_POWER: (no value), con-lstb:MA04-1
- 1R35: device resistor:0207/15 -> resistor:0207/12
- FAN_C: device con-lstb:MA05-2 -> DSS0:MA06-2
- PREH_C: device con-lstb:MA04-2 -> DSS0:MA06-2
- moved 3C14 3.03 mm to (112.2, 160.2)
- moved PREH_C 2.54 mm to (154.5, 100.3)
- moved 3VD10 2.31 mm to (78.1, 119.5)
- moved 3R12 1.63 mm to (87.2, 164.0)
- moved 3C5 1.46 mm to (94.6, 143.0)
- moved FAN_C 1.27 mm to (89.5, 61.9)
- moved 3R6 1.00 mm to (91.4, 149.2)
- moved 3R6B 1.00 mm to (91.4, 149.2)
- moved 1VD11 0.48 mm to (136.4, 64.5)
- moved 1R14 0.32 mm to (133.0, 82.9)
- moved 1R35 0.16 mm to (91.0, 72.1)
Connections:
- net +24V: now also AIR_POWER.1, AIR_POWER.3; no longer AIR.1, R_PW.1
- net GND: now also PREH_C.7, PREH_C.8; no longer PREH_C.5, PREH_C.6
- net M_AIR: now also AIR_POWER.4; no longer AIR.2
- net POWER: now also AIR_POWER.2; no longer R_PW.2
- net TI_PREHEAT: now also PREH_C.10, PREH_C.9; no longer PREH_C.7, PREH_C.8
Routing:
- net M_AIR: track 0.00 -> 3.80 mm
- net GND: track 857.1 -> 853.6 mm
- net IRD: track 14.8 -> 17.2 mm
- net IRVCC: track 74.1 -> 71.8 mm
- net TI_PREHEAT: track 36.3 -> 34.4 mm
- net N$9: track 1.15 -> 2.57 mm
- net PWM_SOL_2: track 76.5 -> 77.7 mm
- net GD: track 14.1 -> 13.0 mm
- net GERKON: track 109.4 -> 110.5 mm
- net ~220V_B: track 111.6 -> 112.7 mm
- net M_FEN: track 94.3 -> 95.3 mm
- net POWER-T: track 177.0 -> 176.0 mm
- net +5V: track 241.8 -> 240.9 mm
- net IROD: track 6.56 -> 7.49 mm
- net D1~I: track 25.3 -> 24.5 mm
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Other:
- board text added: "PREH"
- board text removed: "pr"

Commit message: .
Parts:
- moved 2R5 0.35 mm to (140.7, 170.5)
Routing:
- net POWER-T: track 176.0 -> 185.8 mm
- net POWER-: track 125.1 -> 127.0 mm
